File: 02_Batt_Alim.kicad_pcb (KiCad board)
At the start: 2 copper layers, 29.2 x 25.4 mm, 28 parts, among them IC1 TP4056, J1 Conn_01x01, J2 Conn_01x01, J3 Conn_01x01, J9 Conn_01x01, U1 ME2108A50M3

Commit message: maj librairies
split librairies avec maj chemin, symboles et empreintes + pcb
Parts:
- removed REF**: OSHW-Logo2_7.3x6mm_SilkScreen, Symbol:OSHW-Logo2_7.3x6mm_SilkScreen
- removed REF**: KiCad-Logo2_5mm_SilkScreen, Symbol:KiCad-Logo2_5mm_SilkScreen
- IC1: footprint Chimere:SOP-8 -> Chimere_comps:SOP-8
- J1, J2, J3, J9: footprint Chimere:Castellated_conn -> Chimere_mods:Castellated_conn

Commit message: pcb passage kicad v6
Other:
- net class Default removed
- net class demi-gros removed
- net class gros removed

Commit message: maj schema retouche placement et routage fabrication
Parts:
- D4, D5, D7, D8: value 1N5819W -> SS14; footprint Diode_SMD:D_SOD-123F -> Diode_SMD:D_SMA
- moved C4 7.24 mm to (115.6, 76.7), turned to -90 degrees
- moved R14 6.79 mm to (119.4, 65.5)
- moved D6 3.21 mm to (103.1, 81.5)
- moved C3 2.78 mm to (105.7, 83.8)
- moved U1 2.72 mm to (109.2, 83.3)
- moved D5 2.16 mm to (113.0, 83.1)
- moved D8 1.95 mm to (110.0, 75.4)
- moved R7 1.60 mm to (119.4, 72.1), turned to -90 degrees
- moved D7 1.56 mm to (109.9, 64.8)
- moved R6 1.55 mm to (123.4, 68.7)
- moved D2 1.51 mm to (123.4, 65.5)
- moved R8 1.43 mm to (121.6, 68.7)
- moved D3 1.39 mm to (121.6, 65.5)
- moved L1 1.32 mm to (123.2, 80.5)
- moved C1 1.30 mm to (119.4, 68.9), turned to -90 degrees
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Routing:
- net V_sum: track 27.5 -> 20.6 mm
- net 5V: track 17.2 -> 23.7 mm
- net V_ext: track 38.8 -> 32.4 mm, vias 2 -> 0
- net /V_ext_p: track 15.5 -> 10.4 mm
- net /LX: track 14.6 -> 18.2 mm
- net GND: track 70.7 -> 73.3 mm, vias 13 -> 9
- net V_BAT+: track 18.1 -> 19.7 mm
- net V_chg: track 31.3 -> 29.7 mm
- net Net-(IC1-Pad7): track 20.9 -> 19.4 mm
- net Net-(IC1-Pad6): track 18.8 -> 17.3 mm
- removed copper zone on F.Cu, net /V_ext_p
Other:
- board size 29.2 x 25.4 mm -> 27.9 x 25.4 mm
- board text added: "Batt_Alim_4P 2023/05/10"
- board text removed: "Batt_Alim 2021/02/23"
- board text removed: "github.com/ ThierryOrlandi/ 02_Batt_Alim"
